Commit message: update all files

File: install/smart_car/share/smart_car/urdf/smartcar.urdf.xacro (robot description, xacro)
@@ -2,4 +2,5 @@
 <robot xmlns:xacro="http://www.ros.org/wiki/xacro" name="smart_car">
   <!-- ======================== Parameters ======================== -->
+  <!-- Geometry -->
   <xacro:property name="wheel_diameter" value="0.064"/>
   <xacro:property name="wheel_radius"   value="${wheel_diameter/2.0}"/>
@@ -15,6 +16,10 @@
   <xacro:property name="m_wheel"   value="0.3"/>
   <!-- ========================= Materials ======================== -->
-  <material name="gray"><color rgba="0.6 0.6 0.6 1"/></material>
-  <material name="black"><color rgba="0.1 0.1 0.1 1"/></material>
+  <material name="gray">
+    <color rgba="0.6 0.6 0.6 1"/>
+  </material>
+  <material name="black">
+    <color rgba="0.1 0.1 0.1 1"/>
+  </material>
   <!-- ===================== Inertia Helpers ====================== -->
   <xacro:macro name="inertial_box" params="mass x y z">
@@ -23,6 +28,9 @@
       <origin xyz="0 0 0" rpy="0 0 0"/>
       <inertia
-        ixx="${mass*((y*y+z*z)/12.0)}"  ixy="0" ixz="0"
-        iyy="${mass*((x*x+z*z)/12.0)}"  iyz="0"
+        ixx="${mass*((y*y+z*z)/12.0)}"
+        ixy="0"
+        ixz="0"
+        iyy="${mass*((x*x+z*z)/12.0)}"
+        iyz="0"
         izz="${mass*((x*x+y*y)/12.0)}"/>
     </inertial>
@@ -34,6 +42,9 @@
       <origin xyz="0 0 0" rpy="0 0 0"/>
       <inertia
-        ixx="${mass*((3*r*r+h*h)/12.0)}"  ixy="0" ixz="0"
-        iyy="${mass*((3*r*r+h*h)/12.0)}"  iyz="0"
+        ixx="${mass*((3*r*r+h*h)/12.0)}"
+        ixy="0"
+        ixz="0"
+        iyy="${mass*((3*r*r+h*h)/12.0)}"
+        iyz="0"
         izz="${mass*(r*r/2.0)}"/>
     </inertial>
@@ -50,9 +61,13 @@
   <link name="chassis_link">
     <visual>
-      <geometry><box size="${chassis_len} ${chassis_wid} ${chassis_hei}"/></geometry>
+      <geometry>
+        <box size="${chassis_len} ${chassis_wid} ${chassis_hei}"/>
+      </geometry>
       <material name="gray"/>
     </visual>
     <collision>
-      <geometry><box size="${chassis_len} ${chassis_wid} ${chassis_hei}"/></geometry>
+      <geometry>
+        <box size="${chassis_len} ${chassis_wid} ${chassis_hei}"/>
+      </geometry>
     </collision>
     <xacro:inertial_box mass="${m_chassis}" x="${chassis_len}" y="${chassis_wid}" z="${chassis_hei}"/>
@@ -64,14 +79,19 @@
   </joint>
   <!-- ========================= Wheel Macros ===================== -->
+  <!-- Front: steer joint (about z) → wheel joint (about y) -->
   <xacro:macro name="steered_wheel"
                params="x y steer_joint_name wheel_joint_name steer_link_name wheel_link_name">
     <link name="${steer_link_name}">
       <visual>
-        <geometry><cylinder radius="0.01" length="0.04"/></geometry>
+        <geometry>
+          <cylinder radius="0.01" length="0.04"/>
+        </geometry>
         <origin rpy="1.5708 0 0"/>
         <material name="gray"/>
       </visual>
       <collision>
-        <geometry><cylinder radius="0.01" length="0.04"/></geometry>
+        <geometry>
+          <cylinder radius="0.01" length="0.04"/>
+        </geometry>
         <origin rpy="1.5708 0 0"/>
       </collision>
@@ -86,10 +106,14 @@
     <link name="${wheel_link_name}">
       <visual>
-        <geometry><cylinder radius="${wheel_radius}" length="${wheel_width}"/></geometry>
+        <geometry>
+          <cylinder radius="${wheel_radius}" length="${wheel_width}"/>
+        </geometry>
         <origin rpy="1.5708 0 0"/>
         <material name="black"/>
       </visual>
       <collision>
-        <geometry><cylinder radius="${wheel_radius}" length="${wheel_width}"/></geometry>
+        <geometry>
+          <cylinder radius="${wheel_radius}" length="${wheel_width}"/>
+        </geometry>
         <origin rpy="1.5708 0 0"/>
       </collision>
@@ -102,13 +126,18 @@
     </joint>
   </xacro:macro>
+  <!-- Rear: only wheel joint (about y) -->
   <xacro:macro name="fixed_wheel" params="x y joint_name link_name">
     <link name="${link_name}">
       <visual>
-        <geometry><cylinder radius="${wheel_radius}" length="${wheel_width}"/></geometry>
+        <geometry>
+          <cylinder radius="${wheel_radius}" length="${wheel_width}"/>
+        </geometry>
         <origin rpy="1.5708 0 0"/>
         <material name="black"/>
       </visual>
       <collision>
-        <geometry><cylinder radius="${wheel_radius}" length="${wheel_width}"/></geometry>
+        <geometry>
+          <cylinder radius="${wheel_radius}" length="${wheel_width}"/>
+        </geometry>
         <origin rpy="1.5708 0 0"/>
       </collision>
@@ -128,4 +157,5 @@
   <xacro:property name="y_right" value="${ -wheelbase_wid/2.0 }"/>
   <!-- ===================== Instantiate Wheels =================== -->
+  <!-- Rear -->
   <xacro:fixed_wheel x="${x_back}"  y="${y_left}"
                      joint_name="back_left_wheel_joint"
@@ -134,4 +164,5 @@
                      joint_name="back_right_wheel_joint"
                      link_name="back_right_wheel_link"/>
+  <!-- Front -->
   <xacro:steered_wheel x="${x_front}" y="${y_left}"
                        steer_joint_name="front_left_wheel_steer_joint"
@@ -147,10 +178,14 @@
   <link name="imu_link">
     <visual>
-      <geometry><box size="0.02 0.02 0.02"/></geometry>
+      <geometry>
+        <box size="0.02 0.02 0.02"/>
+      </geometry>
       <origin xyz="0 0 0" rpy="0 0 0"/>
       <material name="gray"/>
     </visual>
     <collision>
-      <geometry><box size="0.02 0.02 0.02"/></geometry>
+      <geometry>
+        <box size="0.02 0.02 0.02"/>
+      </geometry>
       <origin xyz="0 0 0" rpy="0 0 0"/>
     </collision>
@@ -162,5 +197,4 @@
     <child  link="imu_link"/>
   </joint>
-  <!-- Gazebo IMU with RELIABLE QoS -->
   <gazebo reference="imu_link">
     <sensor name="imu_sensor" type="imu">
@@ -172,9 +206,4 @@
           <namespace>/</namespace>
           <remapping>~/out:=/imu_data</remapping>
-          <qos>
-            <reliability>reliable</reliability>
-            <history>keep_last</history>
-            <depth>20</depth>
-          </qos>
         </ros>
         <initial_orientation_as_reference>false</initial_orientation_as_reference>
@@ -185,15 +214,19 @@
   <link name="sllidar_base_link">
     <visual>
-      <geometry><cylinder radius="0.03" length="0.02"/></geometry>
+      <geometry>
+        <cylinder radius="0.03" length="0.02"/>
+      </geometry>
       <origin xyz="0 0 0" rpy="0 0 0"/>
       <material name="black"/>
     </visual>
     <collision>
-      <geometry><cylinder radius="0.03" length="0.02"/></geometry>
+      <geometry>
+        <cylinder radius="0.03" length="0.02"/>
+      </geometry>
       <origin xyz="0 0 0" rpy="0 0 0"/>
     </collision>
     <xacro:inertial_cyl_z mass="0.15" r="0.03" h="0.02"/>
   </link>
-  <!-- Mount the LIDAR at the front; face +X -->
+  <!-- Mount at front; face +X -->
   <joint name="sllidar_mount_joint" type="fixed">
     <origin xyz="${x_front} 0 0.08" rpy="0 0 0"/>
@@ -201,5 +234,4 @@
     <child  link="sllidar_base_link"/>
   </joint>
-  <!-- Gazebo ray sensor: 135° total (±67.5°), centered forward -->
   <gazebo reference="sllidar_base_link">
     <sensor name="front_laser" type="ray">
@@ -210,4 +242,5 @@
         <scan>
           <horizontal>
+            <!-- 135° total FOV, centered forward (±67.5°) -->
             <samples>720</samples>
             <resolution>1</resolution>
@@ -221,5 +254,8 @@
           <resolution>0.01</resolution>
         </range>
-        <noise type="gaussian"><mean>0.0</mean><stddev>0.01</stddev></noise>
+        <noise type="gaussian">
+          <mean>0.0</mean>
+          <stddev>0.01</stddev>
+        </noise>
       </ray>
       <plugin name="gazebo_ros_ray_sensor" filename="libgazebo_ros_ray_sensor.so">
